Commit message: dae file change

File: staubli_tx90_support/urdf/tx_90.urdf (robot description, URDF)
Before this commit: robot staubli_tx90, 11 links, 10 joints
Joints:
- joint joint_6-flange: origin xyz=0 0 0 rpy=0 -1.57079632679 3.1408 -> xyz=0 0 0 rpy=0 -1.57079632679 0
- joint tool_link_fixed: origin xyz=0 0 0 rpy=0 0 0 -> xyz=0 0 0 rpy=0 1.57079632679 0
