Commit message: tool urdf

File: staubli_tx90_support/urdf/tx90_macro.xacro (robot description, xacro)
@@ -157,4 +157,30 @@
                                                  izz="0.000022"/>
       </inertial>
+    </link>
+    <link name="tool_link">
+      <visual>
+        <origin xyz="0 0 0.001" rpy="0 ${radians(-90.0)} ${radians(180.0)}" />
+        <geometry>
+          <mesh filename="package://gripper_2/meshes/base_link.STL" />
+        </geometry>
+        <material name="">
+          <color
+            rgba="0.75294 0.75294 0.75294 1" />
+        </material>
+      </visual>
+      <collision>
+        <origin xyz="0 0 0.005" rpy="0 ${radians(-90.0)} ${radians(180.0)}" />
+        <geometry>
+          <mesh
+            filename="package://gripper_2/meshes/base_link.STL" />
+        </geometry>
+      </collision>
+      <inertial>
+        <mass value="0.00536" />
+        <origin xyz="0.071574 -1.664E-06 0.013015" rpy="0 0 0" />
+        <inertia ixx="0.000012"  ixy="0.0000000"   ixz="0.0000000"
+                                 iyy="0.0013662"   iyz="0.0000000"
+                                                   izz="0.00054605" />
+        </inertial>
     </link>
     <!-- joints: main serial chain -->
@@ -224,9 +250,13 @@
       <child link="${prefix}flange" />
     </joint>
-    <!-- ROS-Industrial 'tool0' frame: all-zeros tool frame -->
+    <joint name="${prefix}tool_link_fixed" type="fixed">
+        <parent link="${prefix}flange"/>
+        <child link="${prefix}tool_link"/>
+        <origin xyz="0 0 0" rpy="0 ${radians(90.0)} 0"/>
+    </joint>
     <link name="${prefix}tool0" />
     <joint name="${prefix}flange-tool0" type="fixed">
-      <origin xyz="0 0 0" rpy="0 ${radians(90.0)} 0" />
-      <parent link="${prefix}flange" />
+      <origin xyz="0.191 0 0.1027" rpy="0 0 0" />
+      <parent link="${prefix}tool_link" />
       <child link="${prefix}tool0" />
     </joint>

Commit message: spindle add

File: staubli_tx90_support/urdf/tx90_macro.xacro (robot description, xacro)
@@ -162,5 +162,5 @@
         <origin xyz="0 0 0.001" rpy="0 ${radians(-90.0)} ${radians(180.0)}" />
         <geometry>
-          <mesh filename="package://gripper_2/meshes/base_link.STL" />
+          <mesh filename="package://spindle/meshes/base_link.STL" />
         </geometry>
         <material name="">
@@ -173,5 +173,5 @@
         <geometry>
           <mesh
-            filename="package://gripper_2/meshes/base_link.STL" />
+            filename="package://spindle/meshes/base_link.STL" />
         </geometry>
       </collision>

Commit message: example works

File: staubli_tx90_support/urdf/tx90_macro.xacro (robot description, xacro)
@@ -257,5 +257,5 @@
     <link name="${prefix}tool0" />
     <joint name="${prefix}flange-tool0" type="fixed">
-      <origin xyz="0.191 0 0.1027" rpy="0 0 0" />
+      <origin xyz="0.191 0 0.1027" rpy="0 ${radians(90.0)} 0" />
       <parent link="${prefix}tool_link" />
       <child link="${prefix}tool0" />
